File: kusabimaru/switches.sch (KiCad schematic (older format))
At the start: 148 parts

Commit message: Exchanged diode footpint to SOD-323
Parts:
- D1, D10, D11, D12, D13, D14, D15, D16, D17, D18, D19, D2, D20, D21, D22, D23, D24, D25, D26, D27, D29, D3, D30, D31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: footprint Diode_SMD:D_0805_2012Metric_Pad1.15x1.40mm_HandSolder -> Diode_SMD:D_SOD-323_HandSoldering
