File: kusabimaru/kuro65.kicad_pcb (KiCad board)
At the start: 2 copper layers, 304.8 x 95.3 mm, 177 parts, among them IC1 ATMEGA32U4, J1 ISP, J2 USB4085-GF-A, SW1 SW_RESET, Y1 16MHz

Commit message: Exchanged old lib folder with kicad_lib repo. Upgraded Kicad files to version 6.
Other:
- net class Default removed
- net class Power removed
- net class USB removed
- net class XTAL removed
