File: kusabimaru/kuro65.kicad_pcb (KiCad board)
At the start: 2 copper layers, 302 x 93 mm, 318 parts, among them IC1 ATMEGA32U4, IC2 ATMEGA32U4, J1 ISP, J2 USB TYPE-C-31-M-12, SW1 SW_RESET, Y1 16MHz

Commit message: Updates in routed PCB.
Parts:
- moved R7 33.5 mm to (104.1, 91.6)
- moved C72 12.5 mm to (4.40, 89.3), turned to 180 degrees
- moved C74 12.5 mm to (52.1, 89.3), turned to 180 degrees
- moved C73 12.4 mm to (28.3, 89.1), turned to 180 degrees
- moved C69 12.2 mm to (242.6, 70.3), turned to 180 degrees
- moved C28 12.1 mm to (30.6, 32.2), turned to 180 degrees
- moved C30 12.1 mm to (68.7, 32.2), turned to 180 degrees
- moved C32 12.1 mm to (106.8, 32.2), turned to 180 degrees
- moved C34 12.1 mm to (144.9, 32.2), turned to 180 degrees
- moved C36 12.1 mm to (183.0, 32.2), turned to 180 degrees
- moved C38 12.1 mm to (221.1, 32.2), turned to 180 degrees
- moved C37 12.0 mm to (202.1, 32.2), turned to 180 degrees
- moved C39 12.0 mm to (240.2, 32.2), turned to 180 degrees
- moved C29 12.0 mm to (49.7, 32.2), turned to 180 degrees
- moved C31 12.0 mm to (87.8, 32.2), turned to 180 degrees
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Connections:
- D101 pad 4: Net-(D101-Pad4) -> Net-(D116-Pad2)
- D117 pad 2: Net-(D117-Pad2) -> Net-(D102-Pad4)
- D118 pad 2: Net-(D117-Pad4) -> Net-(D118-Pad2)
- D131 pad 4: Net-(D116-Pad2) -> Net-(D131-Pad4)
- D132 pad 2: Net-(D132-Pad2) -> Net-(D117-Pad4)
- D132 pad 4: Net-(D117-Pad2) -> Net-(D132-Pad4)
- D133 pad 2: Net-(D133-Pad2) -> Net-(D132-Pad4)
- D133 pad 4: Net-(D132-Pad2) -> Net-(D133-Pad4)
- D134 pad 2: Net-(D134-Pad2) -> Net-(D133-Pad4)
- D134 pad 4: Net-(D133-Pad2) -> Net-(D118-Pad2)
- D135 pad 4: Net-(D134-Pad2) -> /Switches/LED_DI
- D141 pad 2: unconnected-(D141-Pad2) -> Net-(D131-Pad4)
- D38 pad 4: /Switches/LED_DI -> Net-(D87-Pad2)
- D86 pad 2: Net-(D101-Pad4) -> unconnected-(D86-Pad2)
- D87 pad 2: Net-(D102-Pad4) -> Net-(D87-Pad2)
- IC1 pad 1: unconnected-(IC1-Pad1) -> LED_DI
- IC2 pad 1: unconnected-(IC1-Pad1) -> LED_DI
- R7 pad 2: SCK -> LED_DI
Routing:
- net VCC: track 444.8 -> 1752.5 mm, vias 5 -> 9
- net Row3: track 2.32 -> 305.0 mm, vias 0 -> 6
- net Row2: track 2.45 -> 294.3 mm, vias 0 -> 4
- net Row4: track 2.45 -> 293.3 mm, vias 0 -> 6
- net Row1: track 2.57 -> 257.3 mm
- net Row5: track 2.57 -> 164.3 mm
- net Col7: track 3.36 -> 100.0 mm, vias 0 -> 10
- net Col3: track 2.45 -> 95.6 mm, vias 0 -> 6
- net Col2: track 3.36 -> 88.6 mm, vias 0 -> 7
- net Col9: track 2.57 -> 80.1 mm, vias 0 -> 9
- net Col1: track 2.57 -> 79.2 mm, vias 0 -> 6
- net Col8: track 2.70 -> 78.9 mm, vias 0 -> 9
- net Col4: track 2.57 -> 77.1 mm, vias 0 -> 7
- net Col6: track 2.99 -> 76.7 mm, vias 0 -> 9
- net Col5: track 2.70 -> 71.8 mm, vias 0 -> 7
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