File: kusabimaru/kuro65.kicad_sch (KiCad schematic)
At the start: 30 parts, among them IC1 ATMEGA32U4, IC2 ATMEGA32U4, J1 ISP Header, J2 USB TYPE-C-31-M-12, SW1 SW_SPST, Y1 16MHz

Commit message: Updated JLC part numbers in schematic.
Parts:
- C40: LCSC (none) -> C53987; Shop-URL (none) -> https://jlcpcb.com/partdetail/55004-0603B472K500NT/C53987
- R8: LCSC (none) -> C22935; Shop-URL (none) -> https://jlcpcb.com/partdetail/23662-0603WAF1004T5E/C22935
Changed lines of the file:
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@@
       (effects (font (size 1.27 1.27)) hide)
     )
-    (property "Datasheet" "" (id 3) (at 132.715 83.82 0)
+    (property "Datasheet" "https://datasheet.lcsc.com/lcsc/1811061811_FH--Guangdong-Fenghua-Advanced-Tech-0603B472K500NT_C53987.pdf" (id 3) (at 132.715 83.82 0)
       (effects (font (size 1.27 1.27)) hide)
     )
@@
       (effects (font (size 1.27 1.27)) hide)
     )
-    (property "Shop-URL" "" (id 5) (at 132.715 83.82 0)
-      (effects (font (size 1.27 1.27)) hide)
-    )
-    (property "LCSC" "" (id 6) (at 132.715 83.82 0)
+    (property "Shop-URL" "https://jlcpcb.com/partdetail/55004-0603B472K500NT/C53987" (id 5) (at 132.715 83.82 0)
+      (effects (font (size 1.27 1.27)) hide)
+    )
+    (property "LCSC" "C53987" (id 6) (at 132.715 83.82 0)
       (effects (font (size 1.27 1.27)) hide)
     )
@@
       (effects (font (size 1.27 1.27)) hide)
     )
-    (property "Datasheet" "https://datasheet.lcsc.com/lcsc/2206010116_UNI-ROYAL-Uniroyal-Elec-0603WAF5101T5E_C23186.pdf" (id 3) (at 127.635 83.82 0)
+    (property "Datasheet" "https://datasheet.lcsc.com/lcsc/2206010130_UNI-ROYAL-Uniroyal-Elec-0603WAF1004T5E_C22935.pdf" (id 3) (at 127.635 83.82 0)
       (effects (font (size 1.27 1.27)) hide)
     )
@@
       (effects (font (size 1.27 1.27)) hide)
     )
-    (property "Shop-URL" "" (id 5) (at 127.635 83.82 0)
-      (effects (font (size 1.27 1.27)) hide)
-    )
-    (property "LCSC" "" (id 6) (at 127.635 83.82 0)
-      (effects (font (size 1.27 1.27)) hide)
-    )
+    (property "Shop-URL" "https://jlcpcb.com/partdetail/23662-0603WAF1004T5E/C22935" (id 5) (at 127.635 83.82 0)
+      (effects (font (size 1.27 1.27)) hide)
+    )
+    (property "LCSC" "C22935" (id 6) (at 127.635 83.82 0)
+      (effects (font (size 1.27 1.27)) hide)
+    )
